Commit message: update humble

File: urdf/_d435.urdf.xacro (robot description, xacro)
@@ -49,5 +49,5 @@
           <!-- <box size="${d435_cam_width} ${d435_cam_height} ${d435_cam_depth}"/> -->
           <mesh filename="package://realsense2_description/meshes/d435.dae" />
-          <!--<mesh filename="package://realsense2_description/meshes/d435/d435.dae" />-->
+          <!-- <mesh filename="package://husky_description/meshes/accessories/d435.dae" /> -->
         </geometry>
         <material name="${name}_aluminum"/>

File: urdf/test_d435_camera.urdf.xacro (robot description, xacro)
@@ -4,5 +4,5 @@
   <link name="base_link" />
   <xacro:sensor_d435 name="camera" topics_ns="camera" parent="base_link" publish_pointcloud="true">
-    <origin xyz="0 0 0" rpy="0 0 0" />
+    <origin xyz="2 0 2" rpy="0 0 0" />
   </xacro:sensor_d435>
 </robot>

Commit message: fix

File: urdf/_d435.urdf.xacro (robot description, xacro)
@@ -48,6 +48,6 @@
         <geometry>
           <!-- <box size="${d435_cam_width} ${d435_cam_height} ${d435_cam_depth}"/> -->
-          <mesh filename="package://realsense2_description/meshes/d435.dae" />
-          <!-- <mesh filename="package://husky_description/meshes/accessories/d435.dae" /> -->
+          <!-- <mesh filename="package://realsense2_description/meshes/d435.dae" /> -->
+          <mesh filename="package://husky_description/meshes/accessories/d435.dae" />
         </geometry>
         <material name="${name}_aluminum"/>
